Commit message: deleted:    build/r_bot/.cmake/api/v1/query/client-colcon-cmake/codemodel-v2 	deleted:    build/r_bot/.cmake/api/v1/reply/codemodel-v2-761920de8b153622cecc.json 	deleted:    build/r_bot/.cmake/api/v1/reply/directory-.-d5ff0a43bc7e943a0c5c.json 	deleted:    build/r_bot/.cmake/api/v1/reply/index-2026-04-01T09-24-51-0348.json 	deleted:    build/r_bot/.cmake/api/v1/reply/target-r_bot_uninstall-ebd54144b4a6c19a12c2.json 	deleted:    build/r_bot/.cmake/api/v1/reply/target-uninstall-46f8e9cf44eefa20b2d9.json 	deleted:    build/r_bot/CMakeCache.txt 	deleted:    build/r_bot/CMakeFiles/3.22.1/CMakeCCompiler.cmake 	deleted:    build/r_bot/CMakeFiles/3.22.1/CMakeCXXCompiler.cmake 	deleted:    build/r_bot/CMakeFiles/3.22.1/CMakeDetermineCompilerABI_C.bin 	deleted:    build/r_bot/CMakeFiles/3.22.1/CMakeDetermineCompilerABI_CXX.bin 	deleted:    build/r_bot/CMakeFiles/3.22.1/CMakeSystem.cmake 	deleted:    build/r_bot/CMakeFiles/3.22.1/CompilerIdC/CMakeCCompilerId.c 	deleted:    build/r_bot/CMakeFiles/3.22.1/CompilerIdC/a.out 	deleted:    build/r_bot/CMakeFiles/3.22.1/CompilerIdCXX/CMakeCXXCompilerId.cpp 	deleted:    build/r_bot/CMakeFiles/3.22.1/CompilerIdCXX/a.out 	deleted:    build/r_bot/CMakeFiles/CMakeDirectoryInformation.cmake 	deleted:    build/r_bot/CMakeFiles/CMakeOutput.log 	deleted:    build/r_bot/CMakeFiles/CMakeRuleHashes.txt 	deleted:    build/r_bot/CMakeFiles/Makefile.cmake 	deleted:    build/r_bot/CMakeFiles/Makefile2 	deleted:    build/r_bot/CMakeFiles/TargetDirectories.txt 	deleted:    build/r_bot/CMakeFiles/cmake.check_cache 	deleted:    build/r_bot/CMakeFiles/progress.marks 	deleted:    build/r_bot/CMakeFiles/r_bot_uninstall.dir/DependInfo.cmake 	deleted:    build/r_bot/CMakeFiles/r_bot_uninstall.dir/build.make 	deleted:    build/r_bot/CMakeFiles/r_bot_uninstall.dir/cmake_clean.cmake 	deleted:    build/r_bot/CMakeFiles/r_bot_uninstall.dir/compiler_depend.make 	deleted:    build/r_bot/CMakeFiles/r_bot_uninstall.dir/compiler_depend.ts 	deleted:    build/r_bot/CMakeFiles/r_bot_uninstall.dir/progress.make 	deleted:    build/r_bot/CMakeFiles/uninstall.dir/DependInfo.cmake 	deleted:    build/r_bot/CMakeFiles/uninstall.dir/build.make 	deleted:    build/r_bot/CMakeFiles/uninstall.dir/cmake_clean.cmake 	deleted:    build/r_bot/CMakeFiles/uninstall.dir/compiler_depend.make 	deleted:    build/r_bot/CMakeFiles/uninstall.dir/compiler_depend.ts 	deleted:    build/r_bot/CMakeFiles/uninstall.dir/progress.make 	deleted:    build/r_bot/CTestConfiguration.ini 	deleted:    build/r_bot/CTestCustom.cmake 	deleted:    build/r_bot/CTestTestfile.cmake 	deleted:    build/r_bot/Makefile 	deleted:    build/r_bot/ament_cmake_core/package.cmake 	deleted:    build/r_bot/ament_cmake_core/r_botConfig-version.cmake 	deleted:    build/r_bot/ament_cmake_core/r_botConfig.cmake 	deleted:    build/r_bot/ament_cmake_core/stamps/ament_prefix_path.sh.stamp 	deleted:    build/r_bot/ament_cmake_core/stamps/nameConfig-version.cmake.in.stamp 	deleted:    build/r_bot/ament_cmake_core/stamps/nameConfig.cmake.in.stamp 	deleted:    build/r_bot/ament_cmake_core/stamps/package.xml.stamp 	deleted:    build/r_bot/ament_cmake_core/stamps/package_xml_2_cmake.py.stamp 	deleted:    build/r_bot/ament_cmake_core/stamps/path.sh.stamp 	deleted:    build/r_bot/ament_cmake_core/stamps/templates_2_cmake.py.stamp 	deleted:    build/r_bot/ament_cmake_environment_hooks/ament_prefix_path.dsv 	deleted:    build/r_bot/ament_cmake_environment_hooks/local_setup.bash 	deleted:    build/r_bot/ament_cmake_environment_hooks/local_setup.dsv 	deleted:    build/r_bot/ament_cmake_environment_hooks/local_setup.sh 	deleted:    build/r_bot/ament_cmake_environment_hooks/local_setup.zsh 	deleted:    build/r_bot/ament_cmake_environment_hooks/package.dsv 	deleted:    build/r_bot/ament_cmake_environment_hooks/path.dsv 	deleted:    build/r_bot/ament_cmake_index/share/ament_index/resource_index/package_run_dependencies/r_bot 	deleted:    build/r_bot/ament_cmake_index/share/ament_index/resource_index/packages/r_bot 	deleted:    build/r_bot/ament_cmake_index/share/ament_index/resource_index/parent_prefix_path/r_bot 	deleted:    build/r_bot/ament_cmake_package_templates/templates.cmake 	deleted:    build/r_bot/ament_cmake_symlink_install/ament_cmake_symlink_install.cmake 	deleted:    build/r_bot/ament_cmake_symlink_install/ament_cmake_symlink_install_uninstall_script.cmake 	deleted:    build/r_bot/ament_cmake_uninstall_target/ament_cmake_uninstall_target.cmake 	deleted:    build/r_bot/build/lib/r_bot/__init__.py 	deleted:    build/r_bot/build/lib/r_bot/omni_kinematics.py 	deleted:    build/r_bot/cmake_args.last 	deleted:    build/r_bot/cmake_install.cmake 	deleted:    build/r_bot/colcon_command_prefix_build.sh 	deleted:    build/r_bot/colcon_command_prefix_build.sh.env 	modified:   build/r_bot/colcon_command_prefix_setup_py.sh.env 	deleted:    build/r_bot/install.log 	deleted:    build/r_bot/install_manifest.txt 	new file:   build/r_bot/launch/launch_sim.launch.py 	new file:   build/r_bot/launch/new.py 	new file:   build/r_bot/launch/rsp.launch.py 	new file:   build/r_bot/launch/teleop.py 	new file:   build/r_bot/package.xml 	modified:   build/r_bot/prefix_override/__pycache__/sitecustomize.cpython-310.pyc 	new file:   build/r_bot/r_bot 	modified:   build/r_bot/r_bot.egg-info/SOURCES.txt 	new file:   build/r_bot/resource/r_bot 	new file:   build/r_bot/setup.py 	new file:   build/r_bot/share/r_bot/hook/pythonpath_develop.dsv 	new file:   build/r_bot/share/r_bot/hook/pythonpath_develop.ps1 	new file:   build/r_bot/share/r_bot/hook/pythonpath_develop.sh 	deleted:    build/r_bot/symlink_install_manifest.txt 	modified:   install/r_bot/bin/omni_kinematics 	new file:   install/r_bot/lib/python3.10/site-packages/r-bot.egg-link 	deleted:    install/r_bot/lib/python3.10/site-packages/r_bot-0.0.0-py3.10.egg-info/PKG-INFO 	deleted:    install/r_bot/lib/python3.10/site-packages/r_bot-0.0.0-py3.10.egg-info/SOURCES.txt 	deleted:    install/r_bot/lib/python3.10/site-packages/r_bot-0.0.0-py3.10.egg-info/dependency_links.txt 	deleted:    install/r_bot/lib/python3.10/site-packages/r_bot-0.0.0-py3.10.egg-info/entry_points.txt 	deleted:    install/r_bot/lib/python3.10/site-packages/r_bot-0.0.0-py3.10.egg-info/requires.txt 	deleted:    install/r_bot/lib/python3.10/site-packages/r_bot-0.0.0-py3.10.egg-info/top_level.txt 	deleted:    install/r_bot/lib/python3.10/site-packages/r_bot-0.0.0-py3.10.egg-info/zip-safe 	deleted:    install/r_bot/lib/python3.10/site-packages/r_bot/__init__.py 	deleted:    install/r_bot/lib/python3.10/site-packages/r_bot/__pycache__/__init__.cpython-310.pyc 	deleted:    install/r_bot/lib/python3.10/site-packages/r_bot/__pycache__/omni_kinematics.cpython-310.pyc 	deleted:    install/r_bot/share/ament_index/resource_index/package_run_dependencies/r_bot 	typechange: install/r_bot/share/ament_index/resource_index/packages/r_bot 	deleted:    install/r_bot/share/ament_index/resource_index/parent_prefix_path/r_bot 	deleted:    install/r_bot/share/r_bot/cmake/r_botConfig-version.cmake 	deleted:    install/r_bot/share/r_bot/cmake/r_botConfig.cmake 	deleted:    install/r_bot/share/r_bot/config/controllers.yaml 	deleted:    install/r_bot/share/r_bot/config/gui.config 	deleted:    install/r_bot/share/r_bot/config/ros_gz_bridge.yaml 	deleted:    install/r_bot/share/r_bot/config/world.config 	deleted:    install/r_bot/share/r_bot/description/gazebo_control.xacro 	deleted:    install/r_bot/share/r_bot/description/inertial_macro.xacro 	deleted:    install/r_bot/share/r_bot/description/inertial_macros.xacro 	deleted:    install/r_bot/share/r_bot/description/meshes/arm_elbow.dae 	deleted:    install/r_bot/share/r_bot/description/meshes/arm_link.dae 	deleted:    install/r_bot/share/r_bot/description/meshes/base.stl 	deleted:    install/r_bot/share/r_bot/description/meshes/bot.dae 	deleted:    install/r_bot/share/r_bot/description/meshes/bot_marker.png 	deleted:    install/r_bot/share/r_bot/description/meshes/hb_crystal.dae 	deleted:    install/r_bot/share/r_bot/description/meshes/hb_frostbite.dae 	deleted:    install/r_bot/share/r_bot/description/meshes/hb_glacio.dae 	deleted:    install/r_bot/share/r_bot/description/meshes/marker_0.png 	deleted:    install/r_bot/share/r_bot/description/meshes/marker_2.png 	deleted:    install/r_bot/share/r_bot/description/meshes/marker_4.png 	deleted:    install/r_bot/share/r_bot/description/meshes/rim.stl 	deleted:    install/r_bot/share/r_bot/description/meshes/roller.stl 	deleted:    install/r_bot/share/r_bot/description/meshes/wheel.stl 	deleted:    install/r_bot/share/r_bot/description/meshes/wheels.dae 	deleted:    install/r_bot/share/r_bot/description/new_core.xacro 	deleted:    install/r_bot/share/r_bot/description/robot.urdf.xacro 	deleted:    install/r_bot/share/r_bot/description/robot_core copy.xacro 	deleted:    install/r_bot/share/r_bot/description/robot_core.xacro 	deleted:    install/r_bot/share/r_bot/environment/ament_prefix_path.dsv 	deleted:    install/r_bot/share/r_bot/environment/ament_prefix_path.sh 	deleted:    install/r_bot/share/r_bot/environment/path.dsv 	deleted:    install/r_bot/share/r_bot/environment/path.sh 	deleted:    install/r_bot/share/r_bot/hook/cmake_prefix_path.dsv 	deleted:    install/r_bot/share/r_bot/hook/cmake_prefix_path.ps1 	deleted:    install/r_bot/share/r_bot/hook/cmake_prefix_path.sh 	deleted:    install/r_bot/share/r_bot/launch/__pycache__/control.launch.cpython-310.pyc 	deleted:    install/r_bot/share/r_bot/launch/__pycache__/launch_sim.launch.cpython-310.pyc 	deleted:    install/r_bot/share/r_bot/launch/__pycache__/rsp.launch.cpython-310.pyc 	deleted:    install/r_bot/share/r_bot/launch/control.launch.py 	modified:   install/r_bot/share/r_bot/launch/launch_sim.launch.py 	modified:   install/r_bot/share/r_bot/launch/new.py 	modified:   install/r_bot/share/r_bot/launch/rsp.launch.py 	new file:   install/r_bot/share/r_bot/launch/teleop.py 	deleted:    install/r_bot/share/r_bot/local_setup.bash 	deleted:    install/r_bot/share/r_bot/local_setup.dsv 	deleted:    install/r_bot/share/r_bot/local_setup.sh 	deleted:    install/r_bot/share/r_bot/local_setup.zsh 	modified:   install/r_bot/share/r_bot/package.dsv 	modified:   install/r_bot/share/r_bot/package.ps1 	modified:   install/r_bot/share/r_bot/package.sh 	typechange: install/r_bot/share/r_bot/package.xml 	deleted:    log/build_2026-03-22_11-26-37/events.log 	deleted:    log/build_2026-03-22_11-26-37/logger_all.log 	deleted:    log/build_2026-03-22_11-26-37/r_bot/command.log 	deleted:    log/build_2026-03-22_11-26-37/r_bot/stdout.log 	deleted:    log/build_2026-03-22_11-26-37/r_bot/stdout_stderr.log 	deleted:    log/build_2026-03-22_11-26-37/r_bot/streams.log 	deleted:    log/build_2026-03-22_11-31-00/events.log 	deleted:    log/build_2026-03-22_11-31-00/logger_all.log 	deleted:    log/build_2026-03-22_11-31-00/r_bot/command.log 	deleted:    log/build_2026-03-22_11-31-00/r_bot/stdout.log 	deleted:    log/build_2026-03-22_11-31-00/r_bot/stdout_stderr.log 	deleted:    log/build_2026-03-22_11-31-00/r_bot/streams.log 	deleted:    log/build_2026-03-22_11-37-20/events.log 	deleted:    log/build_2026-03-22_11-37-20/logger_all.log 	deleted:    log/build_2026-03-22_11-37-20/r_bot/command.log 	deleted:    log/build_2026-03-22_11-37-20/r_bot/stderr.log 	deleted:    log/build_2026-03-22_11-37-20/r_bot/stdout.log 	deleted:    log/build_2026-03-22_11-37-20/r_bot/stdout_stderr.log 	deleted:    log/build_2026-03-22_11-37-20/r_bot/streams.log 	deleted:    log/build_2026-03-22_11-41-18/events.log 	deleted:    log/build_2026-03-22_11-41-18/logger_all.log 	deleted:    log/build_2026-03-22_11-41-18/r_bot/command.log 	deleted:    log/build_2026-03-22_11-41-18/r_bot/stderr.log 	deleted:    log/build_2026-03-22_11-41-18/r_bot/stdout.log 	deleted:    log/build_2026-03-22_11-41-18/r_bot/stdout_stderr.log 	deleted:    log/build_2026-03-22_11-41-18/r_bot/streams.log 	deleted:    log/build_2026-03-22_11-45-18/events.log 	deleted:    log/build_2026-03-22_11-45-18/logger_all.log 	deleted:    log/build_2026-03-22_11-45-18/r_bot/command.log 	deleted:    log/build_2026-03-22_11-45-18/r_bot/stderr.log 	deleted:    log/build_2026-03-22_11-45-18/r_bot/stdout.log 	deleted:    log/build_2026-03-22_11-45-18/r_bot/stdout_stderr.log 	deleted:    log/build_2026-03-22_11-45-18/r_bot/streams.log 	deleted:    log/build_2026-03-22_11-48-51/events.log 	deleted:    log/build_2026-03-22_11-48-51/logger_all.log 	deleted:    log/build_2026-03-22_11-48-51/r_bot/command.log 	deleted:    log/build_2026-03-22_11-48-51/r_bot/stderr.log 	deleted:    log/build_2026-03-22_11-48-51/r_bot/stdout.log 	deleted:    log/build_2026-03-22_11-48-51/r_bot/stdout_stderr.log 	deleted:    log/build_2026-03-22_11-48-51/r_bot/streams.log 	deleted:    log/build_2026-03-22_11-53-36/events.log 	deleted:    log/build_2026-03-22_11-53-36/logger_all.log 	deleted:    log/build_2026-03-22_11-53-36/r_bot/command.log 	deleted:    log/build_2026-03-22_11-53-36/r_bot/stderr.log 	deleted:    log/build_2026-03-22_11-53-36/r_bot/stdout.log 	deleted:    log/build_2026-03-22_11-53-36/r_bot/stdout_stderr.log 	deleted:    log/build_2026-03-22_11-53-36/r_bot/streams.log 	deleted:    log/build_2026-03-22_11-58-40/events.log 	deleted:    log/build_2026-03-22_11-58-40/logger_all.log 	deleted:    log/build_2026-03-22_11-58-40/r_bot/command.log 	deleted:    log/build_2026-03-22_11-58-40/r_bot/stderr.log 	deleted:    log/build_2026-03-22_11-58-40/r_bot/stdout.log 	deleted:    log/build_2026-03-22_11-58-40/r_bot/stdout_stderr.log 	deleted:    log/build_2026-03-22_11-58-40/r_bot/streams.log 	deleted:    log/build_2026-03-22_12-01-58/events.log 	deleted:    log/build_2026-03-22_12-01-58/logger_all.log 	deleted:    log/build_2026-03-22_12-01-58/r_bot/command.log 	deleted:    log/build_2026-03-22_12-01-58/r_bot/stderr.log 	deleted:    log/build_2026-03-22_12-01-58/r_bot/stdout.log 	deleted:    log/build_2026-03-22_12-01-58/r_bot/stdout_stderr.log 	deleted:    log/build_2026-03-22_12-01-58/r_bot/streams.log 	deleted:    log/build_2026-03-22_12-05-57/events.log 	deleted:    log/build_2026-03-22_12-05-57/logger_all.log 	deleted:    log/build_2026-03-22_12-05-57/r_bot/command.log 	deleted:    log/build_2026-03-22_12-05-57/r_bot/stderr.log 	deleted:    log/build_2026-03-22_12-05-57/r_bot/stdout.log 	deleted:    log/build_2026-03-22_12-05-57/r_bot/stdout_stderr.log 	deleted:    log/build_2026-03-22_12-05-57/r_bot/streams.log 	deleted:    log/build_2026-03-22_20-40-26/events.log 	deleted:    log/build_2026-03-22_20-40-26/logger_all.log 	deleted:    log/build_2026-03-22_20-40-26/r_bot/command.log 	deleted:    log/build_2026-03-22_20-40-26/r_bot/stderr.log 	deleted:    log/build_2026-03-22_20-40-26/r_bot/stdout.log 	deleted:    log/build_2026-03-22_20-40-26/r_bot/stdout_stderr.log 	deleted:    log/build_2026-03-22_20-40-26/r_bot/streams.log 	deleted:    log/build_2026-03-22_20-46-55/events.log 	deleted:    log/build_2026-03-22_20-46-55/logger_all.log 	deleted:    log/build_2026-03-22_20-46-55/r_bot/command.log 	deleted:    log/build_2026-03-22_20-46-55/r_bot/stderr.log 	deleted:    log/build_2026-03-22_20-46-55/r_bot/stdout.log 	deleted:    log/build_2026-03-22_20-46-55/r_bot/stdout_stderr.log 	deleted:    log/build_2026-03-22_20-46-55/r_bot/streams.log 	deleted:    log/build_2026-03-22_20-53-05/events.log 	deleted:    log/build_2026-03-22_20-53-05/logger_all.log 	deleted:    log/build_2026-03-22_20-53-05/r_bot/command.log 	deleted:    log/build_2026-03-22_20-53-05/r_bot/stderr.log 	deleted:    log/build_2026-03-22_20-53-05/r_bot/stdout.log 	deleted:    log/build_2026-03-22_20-53-05/r_bot/stdout_stderr.log 	deleted:    log/build_2026-03-22_20-53-05/r_bot/streams.log 	deleted:    log/build_2026-03-22_20-54-31/events.log 	deleted:    log/build_2026-03-22_20-54-31/logger_all.log 	deleted:    log/build_2026-03-22_20-54-31/r_bot/command.log 	deleted:    log/build_2026-03-22_20-54-31/r_bot/stderr.log 	deleted:    log/build_2026-03-22_20-54-31/r_bot/stdout.log 	deleted:    log/build_2026-03-22_20-54-31/r_bot/stdout_stderr.log 	deleted:    log/build_2026-03-22_20-54-31/r_bot/streams.log 	deleted:    log/build_2026-03-22_20-57-49/events.log 	deleted:    log/build_2026-03-22_20-57-49/logger_all.log 	deleted:    log/build_2026-03-22_20-57-49/r_bot/command.log 	deleted:    log/build_2026-03-22_20-57-49/r_bot/stderr.log 	deleted:    log/build_2026-03-22_20-57-49/r_bot/stdout.log 	deleted:    log/build_2026-03-22_20-57-49/r_bot/stdout_stderr.log 	deleted:    log/build_2026-03-22_20-57-49/r_bot/streams.log 	deleted:    log/build_2026-03-22_20-59-32/events.log 	deleted:    log/build_2026-03-22_20-59-32/logger_all.log 	deleted:    log/build_2026-03-22_20-59-32/r_bot/command.log 	deleted:    log/build_2026-03-22_20-59-32/r_bot/stderr.log 	deleted:    log/build_2026-03-22_20-59-32/r_bot/stdout.log 	deleted:    log/build_2026-03-22_20-59-32/r_bot/stdout_stderr.log 	deleted:    log/build_2026-03-22_20-59-32/r_bot/streams.log 	deleted:    log/build_2026-03-22_21-00-06/events.log 	deleted:    log/build_2026-03-22_21-00-06/logger_all.log 	deleted:    log/build_2026-03-22_21-00-06/r_bot/command.log 	deleted:    log/build_2026-03-22_21-00-06/r_bot/stderr.log 	deleted:    log/build_2026-03-22_21-00-06/r_bot/stdout.log 	deleted:    log/build_2026-03-22_21-00-06/r_bot/stdout_stderr.log 	deleted:    log/build_2026-03-22_21-00-06/r_bot/streams.log 	deleted:    log/build_2026-03-22_21-24-53/events.log 	deleted:    log/build_2026-03-22_21-24-53/logger_all.log 	deleted:    log/build_2026-03-22_21-24-53/r_bot/command.log 	deleted:    log/build_2026-03-22_21-24-53/r_bot/stderr.log 	deleted:    log/build_2026-03-22_21-24-53/r_bot/stdout.log 	deleted:    log/build_2026-03-22_21-24-53/r_bot/stdout_stderr.log 	deleted:    log/build_2026-03-22_21-24-53/r_bot/streams.log 	deleted:    log/build_2026-03-22_21-32-05/events.log 	deleted:    log/build_2026-03-22_21-32-05/logger_all.log 	deleted:    log/build_2026-03-22_21-32-05/r_bot/command.log 	deleted:    log/build_2026-03-22_21-32-05/r_bot/stderr.log 	deleted:    log/build_2026-03-22_21-32-05/r_bot/stdout.log 	deleted:    log/build_2026-03-22_21-32-05/r_bot/stdout_stderr.log 	deleted:    log/build_2026-03-22_21-32-05/r_bot/streams.log 	deleted:    log/build_2026-03-22_21-36-34/events.log 	deleted:    log/build_2026-03-22_21-36-34/logger_all.log 	deleted:    log/build_2026-03-22_21-36-34/r_bot/command.log 	deleted:    log/build_2026-03-22_21-36-34/r_bot/stderr.log 	deleted:    log/build_2026-03-22_21-36-34/r_bot/stdout.log 	deleted:    log/build_2026-03-22_21-36-34/r_bot/stdout_stderr.log 	deleted:    log/build_2026-03-22_21-36-34/r_bot/streams.log 	deleted:    log/build_2026-03-22_21-45-18/events.log 	deleted:    log/build_2026-03-22_21-45-18/logger_all.log 	deleted:    log/build_2026-03-22_21-45-18/r_bot/command.log 	deleted:    log/build_2026-03-22_21-45-18/r_bot/stderr.log 	deleted:    log/build_2026-03-22_21-45-18/r_bot/stdout.log 	deleted:    log/build_2026-03-22_21-45-18/r_bot/stdout_stderr.log 	deleted:    log/build_2026-03-22_21-45-18/r_bot/streams.log 	deleted:    log/build_2026-03-22_21-47-29/events.log 	deleted:    log/build_2026-03-22_21-47-29/logger_all.log 	deleted:    log/build_2026-03-22_21-47-29/r_bot/command.log 	deleted:    log/build_2026-03-22_21-47-29/r_bot/stderr.log 	deleted:    log/build_2026-03-22_21-47-29/r_bot/stdout.log 	deleted:    log/build_2026-03-22_21-47-29/r_bot/stdout_stderr.log 	deleted:    log/build_2026-03-22_21-47-29/r_bot/streams.log 	deleted:    log/build_2026-03-22_21-47-30/events.log 	deleted:    log/build_2026-03-22_21-47-30/logger_all.log 	deleted:    log/build_2026-03-22_21-47-30/r_bot/command.log 	deleted:    log/build_2026-03-22_21-47-30/r_bot/stderr.log 	deleted:    log/build_2026-03-22_21-47-30/r_bot/stdout.log 	deleted:    log/build_2026-03-22_21-47-30/r_bot/stdout_stderr.log 	deleted:    log/build_2026-03-22_21-47-30/r_bot/streams.log 	deleted:    log/build_2026-03-22_21-48-45/events.log 	deleted:    log/build_2026-03-22_21-48-45/logger_all.log

File: src/r_bot/description/original_core_file.xacro (robot description, xacro)
@@ -1,58 +1,56 @@
 <?xml version="1.0"?>
 <robot xmlns:xacro="http://www.ros.org/wiki/xacro" name="hb_bot">
-    <!-- ================= GLOBAL PARAMETERS ================= -->
-    <xacro:property name="wheel_mass" value="0.05"/>
-    <xacro:property name="wheel_radius" value="0.03"/>
-    <xacro:property name="wheel_thickness" value="0.01"/>
-    <!-- ================= INERTIA MACROS ================= -->
+    <!-- Cylinder Inertia: Ixx = Iyy = m*(3r² + h²)/12, Izz = m*r²/2 -->
     <xacro:macro name="cylinder_inertia" params="m r h">
         <inertia
-            ixx="${m*(3*r*r + h*h)/12}" ixy="0" ixz="0"
-            iyy="${m*(3*r*r + h*h)/12}" iyz="0"
-            izz="${m*r*r/2}" />
+        ixx="${m*(3*r*r + h*h)/12}" ixy="0"    ixz="0"
+        iyy="${m*(3*r*r + h*h)/12}" iyz="0"
+        izz="${m*r*r/2}" />
     </xacro:macro>
+    <!-- Box Inertia: Ixx = m*(y²+z²)/12, Iyy = m*(x²+z²)/12, Izz = m*(x²+y²)/12 -->
     <xacro:macro name="box_inertia" params="m x y z">
         <inertia
-            ixx="${m*(y*y + z*z)/12}" ixy="0" ixz="0"
-            iyy="${m*(x*x + z*z)/12}" iyz="0"
-            izz="${m*(x*x + y*y)/12}" />
+        ixx="${m*(y*y + z*z)/12}" ixy="0"    ixz="0"
+        iyy="${m*(x*x + z*z)/12}" iyz="0"
+        izz="${m*(x*x + y*y)/12}" />
     </xacro:macro>
-    <!-- ================= WHEEL MACRO ================= -->
-    <xacro:macro name="rim_macro" params="name xyz rpy mass radius thickness">
+    <xacro:macro name="rim_macro" params="name xyz rpy">
         <link name="rim_${name}_link">
-            <inertial>
-                <origin xyz="0 0 0"/>
-                <mass value="${mass}"/>
-                <xacro:cylinder_inertia m="${mass}" r="${radius}" h="${thickness}"/>
-            </inertial>
-            <visual>
-                <geometry>
-                    <mesh filename="file:///home/deepanshu/My_ROS/src/r_bot/description/meshes/wheels.dae"/>
-                </geometry>
-            </visual>
-            <collision>
-                <geometry>
-                    <cylinder radius="${radius}" length="${thickness}"/>
-                </geometry>
-            </collision>
+        <inertial>
+            <origin xyz="0 0 -0.000343"/>
+            <mass value="0.00835758"/>
+            <inertia ixx="6.63684e-07" ixy="0" ixz="0" iyy="6.63684e-07" iyz="0" izz="9.40333e-07"/>
+        </inertial>
+        <visual>
+            <geometry>
+            <mesh filename="file:///home/deepanshu/My_ROS/src/r_bot/description/meshes/wheels.dae" />
+            </geometry>
+        </visual>
+        <collision>
+            <geometry>
+                <sphere radius="0.016"/>
+            </geometry>
+        </collision>
         </link>
         <joint name="rim_${name}_joint" type="continuous">
-            <parent link="base_link"/>
-            <child link="rim_${name}_link"/>
-            <axis xyz="0 0 1"/>
-            <limit effort="1.0" velocity="10.0"/>
-            <origin xyz="${xyz}" rpy="${rpy}"/>
+        <parent link="base_link"/>
+        <child link="rim_${name}_link"/>
+        <axis xyz="0 0 1"/>
+        <limit effort="1.0" velocity="10.0" lower="-1.79769e+308" upper="1.79769e+308"/>
+        <origin xyz="${xyz}" rpy="${rpy}"/>
         </joint>
     </xacro:macro>
-    <!-- ================= BASE ================= -->
-    <link name="root_link"/>
+    <!-- Root link starts from here -->
+    <link name="root_link">
+    </link>
     <link name="base_link">
         <visual>
+            <origin xyz="0 0 0" rpy="0 0 0" />
             <geometry>
                 <mesh filename="file:///home/deepanshu/My_ROS/src/r_bot/description/meshes/hb_crystal.dae"/>
             </geometry>
         </visual>
-        <collision>
-            <origin xyz="0 0 0.042"/>
+        <collision name="base_link_collision">
+            <origin xyz="0 0 0.042" rpy="0 0 0" />
             <geometry>
                 <cylinder length="0.064" radius="0.08"/>
@@ -60,7 +58,7 @@
         </collision>
         <inertial>
-            <origin xyz="0 0 0"/>
-            <mass value="0.15"/>
-            <xacro:cylinder_inertia m="0.15" r="0.074" h="0.03"/>
+            <origin xyz="0 0 0" rpy="0 0 0" />
+            <mass value="0.15" />
+            <xacro:cylinder_inertia m="0.3" r="0.074" h="0.03"/>
         </inertial>
     </link>
@@ -68,16 +66,19 @@
         <parent link="root_link"/>
         <child link="base_link"/>
+        <origin xyz="0 0 0" rpy="0 0 0" />
     </joint>
-    <!-- ================= ARM ================= -->
-    <link name="chassis_link"/>
-    <link name="arm_root_link"/>
+    <link name="chassis_link">
+    </link>
+    <link name="arm_root_link">
+    </link>
     <link name="arm_link_1">
         <visual>
+            <origin xyz="0 0 0" rpy="0 0 0" />
             <geometry>
                 <mesh filename="file:///home/deepanshu/My_ROS/src/r_bot/description/meshes/arm_link.dae"/>
             </geometry>
         </visual>
-        <collision>
-            <origin xyz="0 0 0.02472"/>
+        <collision name="arm_link_1_collision">
+            <origin xyz="0 0 0.02472" rpy="0 0 0" />
             <geometry>
                 <box size="0.008 0.008 0.06"/>
@@ -85,5 +86,6 @@
         </collision>
         <inertial>
-            <mass value="0.001"/>
+            <origin xyz="0 0 0" rpy="0 0 0" />
+            <mass value="0.001" />
             <xacro:cylinder_inertia m="0.001" r="0.025" h="0.05"/>
         </inertial>
@@ -91,10 +93,11 @@
     <link name="arm_link_2">
         <visual>
+            <origin xyz="0 0 0" rpy="0 0 0" />
             <geometry>
                 <mesh filename="file:///home/deepanshu/My_ROS/src/r_bot/description/meshes/arm_elbow.dae"/>
             </geometry>
         </visual>
-        <collision>
-            <origin xyz="0 0 0.025"/>
+        <collision name="arm_link_2_collision">
+            <origin xyz="0 0 0.025" rpy="0 0 0" />
             <geometry>
                 <box size="0.008 0.008 0.05"/>
@@ -102,52 +105,37 @@
         </collision>
         <inertial>
-            <mass value="0.001"/>
+            <origin xyz="0 0 0" rpy="0 0 0" />
+            <mass value="0.001" />
             <xacro:cylinder_inertia m="0.001" r="0.025" h="0.05"/>
         </inertial>
     </link>
-    <!-- Fixed arm chain -->
     <joint name="base_to_chassis" type="fixed">
         <parent link="base_link"/>
         <child link="chassis_link"/>
-        <origin xyz="0 0 0.0795"/>
+        <origin xyz="0 0 0.0795" rpy="0 0 0" />
     </joint>
     <joint name="chassis_to_arm_base" type="fixed">
         <parent link="chassis_link"/>
         <child link="arm_root_link"/>
-        <origin xyz="0.075 0 0"/>
+        <origin xyz="0.075 0 0" rpy="0 0 0" />
     </joint>
     <joint name="arm_base" type="fixed">
         <parent link="arm_root_link"/>
         <child link="arm_link_1"/>
-        <origin xyz="0 0 0.013"/>
+        <origin xyz="0 0 0.013" rpy="0 0 0" />
+        <axis xyz="0 1 0"/>
+        <limit effort="1.0" velocity="2.0" lower="-3.14" upper="3.14"/>
     </joint>
     <joint name="arm_elbow" type="fixed">
         <parent link="arm_link_1"/>
         <child link="arm_link_2"/>
-        <origin xyz="0 0 0.05"/>
+        <origin xyz="0 0 0.05" rpy="0 0 0" />
+        <axis xyz="0 1 0"/>
+        <limit effort="1.0" velocity="2.0" lower="-3.14" upper="3.14"/>
     </joint>
-    <!-- ================= WHEELS ================= -->
-    <xacro:rim_macro
-        name="left"
-        xyz="0.03600001399230441 0.06235382099401676 -0.001"
-        rpy="1.570796326794896 0 -0.523599"
-        mass="${wheel_mass}"
-        radius="${wheel_radius}"
-        thickness="${wheel_thickness}"/>
-    <xacro:rim_macro
-        name="right"
-        xyz="0.03600001399230441 -0.06235382099401676 -0.001"
-        rpy="1.570796326794896 0 0.523599"
-        mass="${wheel_mass}"
-        radius="${wheel_radius}"
-        thickness="${wheel_thickness}"/>
-    <xacro:rim_macro
-        name="back"
-        xyz="-0.072 0 0"
-        rpy="1.570796326794896 0 1.570796326794896"
-        mass="${wheel_mass}"
-        radius="${wheel_radius}"
-        thickness="${wheel_thickness}"/>
-    <!-- ================= CONTROL ================= -->
+    <!-- the wheels are here -->
+    <xacro:rim_macro name="left" xyz="0.03600001399230441 0.06235382099401676 -0.001" rpy="1.570796326794896 0 -0.523599"/>
+    <xacro:rim_macro name="right" xyz="0.03600001399230441 -0.06235382099401676 -0.001"  rpy="1.570796326794896 0 0.523599"/>
+    <xacro:rim_macro name="back" xyz="-0.072 0 0" rpy="1.570796326794896 0 1.570796326794896"/>
     <ros2_control name="RobotSystem" type="system">
         <hardware>
@@ -170,5 +158,4 @@
         </joint>
     </ros2_control>
-    <!-- ================= GAZEBO ================= -->
     <gazebo>
         <plugin name="gazebo_ros2_control" filename="libgazebo_ros2_control.so">
