Commit message: renamed:    build/r_bot/.cmake/api/v1/reply/index-2026-05-07T19-13-54-0916.json -> build/r_bot/.cmake/api/v1/reply/index-2026-05-08T17-30-22-0181.json 	modified:   build/r_bot/cmake_args.last 	modified:   build/r_bot/colcon_command_prefix_build.sh.env 	modified:   build/r_bot/symlink_install_manifest.txt 	new file:   install/r_bot/share/r_bot/config/mapper_params_online_async.yaml 	modified:   install/r_bot/share/r_bot/hook/path.ps1 	modified:   install/r_bot/share/r_bot/hook/pythonpath.ps1 	modified:   install/r_bot/share/r_bot/hook/pythonscriptspath.ps1 	modified:   install/r_bot/share/r_bot/package.ps1 	modified:   install/setup.ps1 	new file:   log/build_2026-05-08_22-53-50/events.log 	new file:   log/build_2026-05-08_22-53-50/logger_all.log 	new file:   log/build_2026-05-08_22-53-50/r_bot/command.log 	new file:   log/build_2026-05-08_22-53-50/r_bot/stderr.log 	new file:   log/build_2026-05-08_22-53-50/r_bot/stdout.log 	new file:   log/build_2026-05-08_22-53-50/r_bot/stdout_stderr.log 	new file:   log/build_2026-05-08_22-53-50/r_bot/streams.log 	new file:   log/build_2026-05-08_23-00-21/events.log 	new file:   log/build_2026-05-08_23-00-21/logger_all.log 	new file:   log/build_2026-05-08_23-00-21/r_bot/command.log 	new file:   log/build_2026-05-08_23-00-21/r_bot/stderr.log 	new file:   log/build_2026-05-08_23-00-21/r_bot/stdout.log 	new file:   log/build_2026-05-08_23-00-21/r_bot/stdout_stderr.log 	new file:   log/build_2026-05-08_23-00-21/r_bot/streams.log 	new file:   log/build_2026-05-08_23-28-28/events.log 	new file:   log/build_2026-05-08_23-28-28/logger_all.log 	new file:   log/build_2026-05-08_23-28-28/r_bot/command.log 	new file:   log/build_2026-05-08_23-28-28/r_bot/stderr.log 	new file:   log/build_2026-05-08_23-28-28/r_bot/stdout.log 	new file:   log/build_2026-05-08_23-28-28/r_bot/stdout_stderr.log 	new file:   log/build_2026-05-08_23-28-28/r_bot/streams.log 	modified:   log/latest_build 	new file:   src/r_bot/config/mapper_params_online_async.yaml 	modified:   src/r_bot/description/new_core.xacro 	new file:   src/r_bot/worlds/obstacles_main

File: src/r_bot/description/new_core.xacro (robot description, xacro)
@@ -69,4 +69,12 @@
         <child link="base_link"/>
     </joint>
+    <!-- BASE_FOOTPRINT LINK -->
+    <joint name="base_footprint_joint" type="fixed">
+        <parent link="base_link"/>
+        <child link="base_footprint"/>
+        <origin xyz="0 0 0" rpy="0 0 0"/>
+    </joint>
+    <link name="base_footprint">
+    </link>
     <!-- ================= ARM ================= -->
     <link name="chassis_link"/>
